File: main.kicad_pcb (KiCad board)
At the start: 4 copper layers, 228.6 x 70.6 mm, 141 parts, among them J1 Conn_02x16_Row_Letter_First, J10 Conn_01x26_Pin, J2 Conn_01x03, J4 Screw_Terminal_01x02, J5 Screw_Terminal_01x10, J6 Screw_Terminal_01x10, J7 Screw_Terminal_01x02, J8 Screw_Terminal_01x10, J9 Screw_Terminal_01x10, U1 SN74ACT595, U10 AQY216EH, U11 AQY216EH, U12 AQY216EH, U13 AQY216EH, U14 AQY216EH, U15 AQY216EH, U16 AQY216EH, U17 AQY216EH, U18 AQY216EH, U19 AQY216EH, U2 SN74ACT595, U20 AQY216EH, U21 AQY216EH, U22 AQY216EH, U23 AQY216EH, U24 AQY216EH, U25 AQY216EH, U26 AQY216EH, U27 AQY216EH, U28 AQY216EH, U29 AQY216EH, U3 74HC74, U30 AQY216EH, U31 AQY216EH, U32 AQY216EH, U33 AQY216EH, U34 AQY216EH, U35 AQY216EH, U36 AQY216EH, U37 AQY216EH, U38 AQY216EH, U39 AQY216EH, U4 AQY216EH, U40 AQY216EH, U41 AQY216EH, U42 AQY216EH, U43 AQY216EH, U44 AQY216EH, U45 AQY216EH, U46 AQY216EH, U47 AQY216EH, U48 TL7705AxPS, U49 SN74ACT595, U5 AQY216EH, U50 74AHC1G04, U51 74AHC1G08, U52 74AHC1G04, U53 TLV7012DSGR, U6 AQY216EH, U7 AQY216EH, U8 AQY216EH, U9 AQY216EH

Commit message: Added Image
Other:
- board text added: "ID"
- board text added: "~{RST}"
