File: mcu.kicad_sch (KiCad schematic)
At the start: 29 parts, among them U1 SN74ACT595, U2 SN74ACT595, U3 74HC74, U48 TL7705AxPS, U49 SN74ACT595, U50 74AHC1G04, U51 74AHC1G08, U52 74AHC1G04, U53 TLV7012DSGR

Commit message: Added Image
Parts:
- U48: value TL7705AxPS -> TL7705ACPS
Changed lines of the file:
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@@
 			)
 		)
-		(property "Value" "TL7705AxPS"
+		(property "Value" "TL7705ACPS"
 			(at 58.0233 80.01 0)
 			(effects
@@
 					(reference "U48")
 					(unit 1)
+				)
+				(path "/29195ea4-8218-44a1-b4bf-466bee0082e4/00000000-0000-0000-0000-000061fc209f"
+					(reference "U48")
+					(unit 1)
